File: LEVIA_H7.kicad_pcb (KiCad board)
At the start: 6 copper layers, 39.5 x 39.5 mm, 158 parts, among them J1 TF-028-H265, Q1 AO3400A, SW2 RKCGG140SMTRLFS, U1 USBLC6-2P6, U10 ZX-SH1.0-4PWT, U11 ZX-SH1.0-3PWT, U12 SIT1051TK/3, U13 ZX-SH1.0-4PWT, U14 ICM-42688-P, U15 ICM-42688-P, U16 DPS368XTSA1, U17 IST8310, U18 ZX-SH1.0-4PWT, U19 ZX-SH1.0-6PWT, U2 STM32H743VIHx, U20 ZX-SH1.0-6PWT, U21 ZX-SH1.0-3PWT, U22 ZX-SH1.0-8PWT, U24 ZX-SH1.0-4PWT, U3 ZX-SH1.0-4PWT, U4 LMR43620R5RPER, U5 LMR604303SRAKRQ1, U6 AP7361C-33FGE-7, U7 AP7361C-33FGE-7, U8 ZX-SH1.0-4PWT, U9 AT7456ELAH, Y1 8MHz, Y2 XL7EL89COI-111YLC-27M

Commit message: b fab layer text edit
Parts:
- turned TP10 to 180 degrees
- turned TP5 to 180 degrees
- turned TP6 to 180 degrees
- turned TP7 to 180 degrees
- turned TP8 to 180 degrees
- turned TP9 to 180 degrees
Changed lines of the file:
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@@
 		)
 		(fp_text user "${REFERENCE}"
-			(at 0 2.5 135)
+			(at -0.014142 0.014142 135)
 			(unlocked yes)
 			(layer "F.Fab")
@@
 			(unlocked yes)
 			(layer "B.SilkS")
+			(hide yes)
 			(effects
 				(font
@@
 		)
 		(fp_text user "${REFERENCE}"
-			(at 0 1.74 0)
+			(at 0 0.019383 90)
 			(unlocked yes)
 			(layer "B.Fab")
@@
 	(footprint "EasyEDA:TestPoint_Pad_1.8x0.9mm"
 		(layer "B.Cu")
-		(at 139.919995 51.425004)
+		(at 139.919995 51.425004 180)
 		(descr "SMD rectangular pad as test Point, square 1.0mm side length")
 		(tags "test point SMD pad rectangle square")
 		(property "Reference" "TP8"
-			(at 0.01 1.62 0)
+			(at 0.01 1.62 180)
 			(unlocked yes)
 			(layer "B.SilkS")
+			(hide yes)
 			(effects
 				(font
@@
 		)
 		(property "Datasheet" ""
-			(at 0 0 180)
+			(at 0 0 0)
 			(unlocked yes)
 			(layer "B.Fab")
@@
 		)
 		(property "Description" "test point"
-			(at 0 0 180)
+			(at 0 0 0)
 			(unlocked yes)
 			(layer "B.Fab")
@@
 		)
 		(fp_text user "${REFERENCE}"
-			(at 0 1.74 0)
+			(at 0 0.019383 90)
 			(unlocked yes)
 			(layer "B.Fab")
@@
 		)
 		(pad "1" smd roundrect
-			(at 0 0)
+			(at 0 0 180)
 			(size 0.9 1.8)
 			(layers "B.Cu" "B.Mask")
@@
 	(footprint "EasyEDA:TestPoint_Pad_1.8x0.9mm"
 		(layer "B.Cu")
-		(at 143.959283 51.400004)
+		(at 143.959283 51.400004 180)
 		(descr "SMD rectangular pad as test Point, square 1.0mm side length")
 		(tags "test point SMD pad rectangle square")
 		(property "Reference" "TP5"
-			(at 0.01 1.62 0)
+			(at 0.01 1.62 180)
 			(unlocked yes)
 			(layer "B.SilkS")
+			(hide yes)
 			(effects
 				(font
@@
 		)
 		(property "Datasheet" ""
-			(at 0 0 180)
+			(at 0 0 0)
 			(unlocked yes)
 			(layer "B.Fab")
@@
 		)
 		(property "Description" "test point"
-			(at 0 0 180)
+			(at 0 0 0)
 			(unlocked yes)
 			(layer "B.Fab")
@@
 		)
 		(fp_text user "${REFERENCE}"
-			(at 0 1.74 0)
+			(at 0 0.019383 90)
 			(unlocked yes)
 			(layer "B.Fab")
@@
 		)
 		(pad "1" smd roundrect
-			(at 0 0)
+			(at 0 0 180)
 			(size 0.9 1.8)
 			(layers "B.Cu" "B.Mask")
@@
 			(unlocked yes)
 			(layer "B.SilkS")
+			(hide yes)
 			(effects
 				(font
@@
 		)
 		(fp_text user "${REFERENCE}"
-			(at 0 1.74 0)
+			(at 0 0.019383 90)
 			(unlocked yes)
 			(layer "B.Fab")
@@
 			(unlocked yes)
 			(layer "B.SilkS")
+			(hide yes)
 			(effects
 				(font
@@
 		)
 		(fp_text user "${REFERENCE}"
-			(at 0 1.74 0)
+			(at 0 0.019383 90)
 			(unlocked yes)
 			(layer "B.Fab")
@@
 	(footprint "EasyEDA:TestPoint_Pad_1.8x0.9mm"
 		(layer "B.Cu")
-		(at 149.345 51.4)
+		(at 149.345 51.4 180)
 		(descr "SMD rectangular pad as test Point, square 1.0mm side length")
 		(tags "test point SMD pad rectangle square")
 		(property "Reference" "TP9"
-			(at 0.01 1.62 180)
+			(at 0.01 1.62 0)
 			(unlocked yes)
 			(layer "B.SilkS")
+			(hide yes)
 			(effects
 				(font
@@
 		)
 		(property "Value" "~"
-			(at 0 -1.550001 180)
+			(at 0 -1.550001 0)
 			(unlocked yes)
 			(layer "B.Fab")
@@
 		)
 		(property "Datasheet" ""
-			(at 0 0 180)
+			(at 0 0 0)
 			(unlocked yes)
 			(layer "B.Fab")
@@
 		)
 		(property "Description" "test point"
-			(at 0 0 180)
+			(at 0 0 0)
 			(unlocked yes)
 			(layer "B.Fab")
@@
 		)
 		(duplicate_pad_numbers_are_jumpers no)
-		(fp_rect
-			(start -0.52 0.96701)
-			(end 0.52 -0.97)
+		(fp_poly
+			(pts
+				(xy -0.52 -0.97) (xy 0.52 -0.97) (xy 0.52 0.96701) (xy -0.52 0.96701)
+			)
 			(stroke
 				(width 0.02)
@@
 		)
 		(fp_text user "${REFERENCE}"
-			(at 0 1.74 180)
+			(at 0 0.019383 90)
 			(unlocked yes)
 			(layer "B.Fab")
@@
 		)
 		(pad "1" smd roundrect
-			(at 0 0)
+			(at 0 0 180)
 			(size 0.9 1.8)
 			(layers "B.Cu" "B.Mask")
@@
 			(unlocked yes)
 			(layer "B.SilkS")
+			(hide yes)
 			(effects
 				(font
@@
 		)
 		(fp_text user "${REFERENCE}"
-			(at 0 1.74 0)
+			(at 0 0.019383 90)
 			(unlocked yes)
 			(layer "B.Fab")
@@
 			(unlocked yes)
 			(layer "B.SilkS")
+			(hide yes)
 			(effects
 				(font
@@
 		)
 		(fp_text user "${REFERENCE}"
-			(at 0 1.74 0)
+			(at 0 0.019383 90)
 			(unlocked yes)
 			(layer "B.Fab")
@@
 			(unlocked yes)
 			(layer "B.SilkS")
+			(hide yes)
 			(effects
 				(font
@@
 		)
 		(fp_text user "${REFERENCE}"
-			(at 0 1.74 0)
+			(at 0 0.019383 90)
 			(unlocked yes)
 			(layer "B.Fab")
@@
 	(footprint "EasyEDA:TestPoint_Pad_1.8x0.9mm"
 		(layer "B.Cu")
-		(at 142.612854 51.400004)
+		(at 142.612854 51.400004 180)
 		(descr "SMD rectangular pad as test Point, square 1.0mm side length")
 		(tags "test point SMD pad rectangle square")
 		(property "Reference" "TP6"
-			(at 0.01 1.62 0)
+			(at 0.01 1.62 180)
 			(unlocked yes)
 			(layer "B.SilkS")
+			(hide yes)
 			(effects
 				(font
@@
 		)
 		(property "Datasheet" ""
-			(at 0 0 180)
+			(at 0 0 0)
 			(unlocked yes)
 			(layer "B.Fab")
@@
 		)
 		(property "Description" "test point"
-			(at 0 0 180)
+			(at 0 0 0)
 			(unlocked yes)
 			(layer "B.Fab")
@@
 		)
 		(fp_text user "${REFERENCE}"
-			(at 0 1.74 0)
+			(at 0 0.019383 90)
 			(unlocked yes)
 			(layer "B.Fab")
@@
 		)
 		(pad "1" smd roundrect
-			(at 0 0)
+			(at 0 0 180)
 			(size 0.9 1.8)
 			(layers "B.Cu" "B.Mask")
@@
 			(unlocked yes)
 			(layer "B.SilkS")
+			(hide yes)
 			(effects
 				(font
@@
 		)
 		(fp_text user "${REFERENCE}"
-			(at 0 1.74 0)
+			(at 0 0.019383 90)
 			(unlocked yes)
 			(layer "B.Fab")
@@
 	(footprint "EasyEDA:TestPoint_Pad_1.8x0.9mm"
 		(layer "B.Cu")
-		(at 147.998571 51.4)
+		(at 147.998571 51.4 180)
 		(descr "SMD rectangular pad as test Point, square 1.0mm side length")
 		(tags "test point SMD pad rectangle square")
 		(property "Reference" "TP10"
-			(at 0.01 1.62 180)
+			(at 0.01 1.62 0)
 			(unlocked yes)
 			(layer "B.SilkS")
+			(hide yes)
 			(effects
 				(font
@@
 		)
 		(property "Value" "~"
-			(at 0 -1.550001 180)
+			(at 0 -1.550001 0)
 			(unlocked yes)
 			(layer "B.Fab")
@@
 		)
 		(property "Datasheet" ""
-			(at 0 0 180)
+			(at 0 0 0)
 			(unlocked yes)
 			(layer "B.Fab")
@@
 		)
 		(property "Description" "test point"
-			(at 0 0 180)
+			(at 0 0 0)
 			(unlocked yes)
 			(layer "B.Fab")
@@
 		)
 		(duplicate_pad_numbers_are_jumpers no)
-		(fp_rect
-			(start -0.52 0.96701)
-			(end 0.52 -0.97)
+		(fp_poly
+			(pts
+				(xy -0.52 -0.97) (xy 0.52 -0.97) (xy 0.52 0.96701) (xy -0.52 0.96701)
+			)
 			(stroke
 				(width 0.02)
@@
 		)
 		(fp_text user "${REFERENCE}"
-			(at 0 1.74 180)
+			(at 0 0.019383 90)
 			(unlocked yes)
 			(layer "B.Fab")
@@
 		)
 		(pad "1" smd roundrect
-			(at 0 0)
+			(at 0 0 180)
 			(size 0.9 1.8)
 			(layers "B.Cu" "B.Mask")
@@
 			(unlocked yes)
 			(layer "B.SilkS")
+			(hide yes)
 			(effects
 				(font
@@
 		)
 		(duplicate_pad_numbers_are_jumpers no)
-		(fp_rect
-			(start -0.52 0.96701)
-			(end 0.52 -0.97)
+		(fp_poly
+			(pts
+				(xy 0.52 0.96701) (xy -0.52 0.96701) (xy -0.52 -0.97) (xy 0.52 -0.97)
+			)
 			(stroke
 				(width 0.02)
@@
 		)
 		(fp_text user "${REFERENCE}"
-			(at 0 1.74 0)
+			(at 0 0.019383 90)
 			(unlocked yes)
 			(layer "B.Fab")
@@
 			(unlocked yes)
 			(layer "B.SilkS")
+			(hide yes)
 			(effects
 				(font
@@
 		)
 		(fp_text user "${REFERENCE}"
-			(at 0 1.74 0)
+			(at 0 0.019383 90)
 			(unlocked yes)
 			(layer "B.Fab")
@@
 			(unlocked yes)
 			(layer "B.SilkS")
+			(hide yes)
 			(effects
 				(font
@@
 		)
 		(fp_text user "${REFERENCE}"
-			(at 0 1.74 0)
+			(at 0 0.019383 90)
 			(unlocked yes)
 			(layer "B.Fab")
@@
 	(footprint "EasyEDA:TestPoint_Pad_1.8x0.9mm"
 		(layer "B.Cu")
-		(at 141.266424 51.400004)
+		(at 141.266424 51.400004 180)
 		(descr "SMD rectangular pad as test Point, square 1.0mm side length")
 		(tags "test point SMD pad rectangle square")
 		(property "Reference" "TP7"
-			(at 0.01 1.62 0)
+			(at 0.01 1.62 180)
 			(unlocked yes)
 			(layer "B.SilkS")
+			(hide yes)
 			(effects
 				(font
@@
 		)
 		(property "Datasheet" ""
-			(at 0 0 180)
+			(at 0 0 0)
 			(unlocked yes)
 			(layer "B.Fab")
@@
 		)
 		(property "Description" "test point"
-			(at 0 0 180)
+			(at 0 0 0)
 			(unlocked yes)
 			(layer "B.Fab")
@@
 		)
 		(fp_text user "${REFERENCE}"
-			(at 0 1.74 0)
+			(at 0 0.019383 90)
 			(unlocked yes)
 			(layer "B.Fab")
@@
 		)
 		(pad "1" smd roundrect
-			(at 0 0)
+			(at 0 0 180)
 			(size 0.9 1.8)
 			(layers "B.Cu" "B.Mask")

Commit message: save
Parts:
- moved C42 0.95 mm to (147.7, 83.8), turned to 90 degrees
Routing:
- net GND: track 46.7 -> 59.8 mm, vias 116 -> 176
- net Net-(U5-FB): track 0.00 -> 2.96 mm
- net +3V3_MCU: track 108.8 -> 111.0 mm, vias 14 -> 16
- net Net-(U5-MODE/SYNC): track 0.00 -> 1.82 mm
- net /POWER/DJI_EN: track 0.00 -> 1.33 mm
- net /MCU/UART8.RX: track 74.5 -> 73.3 mm
- net /MCU/ADC1_CURR1: track 66.8 -> 65.6 mm
- net Net-(U6-EN): track 0.00 -> 1.13 mm
- net Net-(U5-BOOT): track 0.00 -> 1.05 mm
- net Net-(U5-PG): track 0.00 -> 1.05 mm
- net /CAN/CAN1.SILENT: track 42.2 -> 43.1 mm
- added copper zone on B.Cu, net /POWER/SW_9V

Commit message: labels
Parts:
- added kibuzzard-6A40F422: G***, kibuzzard-6A40F422, F.Cu at (150.6, 62.7)
- added kibuzzard-6A40F45A: G***, kibuzzard-6A40F45A, F.Cu at (151.7, 72.2)
- added kibuzzard-6A40F4B5: G***, kibuzzard-6A40F4B5, F.Cu at (150.7, 80.1)
- added kibuzzard-6A40F56A: G***, kibuzzard-6A40F56A, F.Cu at (145.3, 56.6)
- added kibuzzard-6A40F5CA: G***, kibuzzard-6A40F5CA, B.Cu at (144.6, 53.2)
- added kibuzzard-6A40F62C: G***, kibuzzard-6A40F62C, B.Cu at (135.7, 53.2)
- added kibuzzard-6A40F649: G***, kibuzzard-6A40F649, B.Cu at (130.3, 55.0)
- added kibuzzard-6A40F691: G***, kibuzzard-6A40F691, B.Cu at (126.7, 70.8)
- added kibuzzard-6A40F712: G***, kibuzzard-6A40F712, B.Cu at (126.8, 77.2)
- added kibuzzard-6A40F8CE: G***, kibuzzard-6A40F8CE, B.Cu at (130.9, 80.9)
- added kibuzzard-6A40F981: G***, kibuzzard-6A40F981, B.Cu at (140.9, 81.0)
- added kibuzzard-6A40F9B9: G***, kibuzzard-6A40F9B9, B.Cu at (147.5, 81.0)
- R19, R20: value 100K -> 10K
- moved R32 3.33 mm to (129.3, 78.4), turned to 90 degrees
- moved REF** 0.53 mm to (142.9, 76.2)
- moved C2 0.34 mm to (137.9, 78.2)
- moved C4 0.33 mm to (137.8, 79.2)
- moved R34 0.31 mm to (127.4, 79.8)
- moved R35 0.23 mm to (127.0, 81.3)
- moved C6 0.18 mm to (133.9, 79.0)
- moved C9 0.16 mm to (136.4, 77.2)
- moved D2 0.12 mm to (153.4, 57.9)
- moved C10 0.10 mm to (136.4, 76.1)
- moved C34 0.07 mm to (144.7, 64.6)
- moved C3 0.06 mm to (136.3, 80.7)
Routing:
- net /I2C1|SPI3/SPI3.MOSI: track 14.5 -> 10.6 mm
- net GND: track 59.8 -> 63.2 mm, vias 176 -> 237
- net +5V_SYS: track 183.2 -> 185.2 mm, vias 19 -> 21
- net /MCU/VDD: track 50.2 -> 50.9 mm
- net /I2C1|SPI3/SPI3.MISO: track 9.72 -> 9.02 mm
- net /MCU/ADC1_CURR1: track 65.6 -> 66.2 mm
- added copper zone on In2.Cu, net +5V
- added copper zone on F.Cu, net +5V_SYS

Commit message: first drc pass
Parts:
- moved NT1 0.84 mm to (128.5, 58.5), turned to -135 degrees
- moved R40 0.30 mm to (130.6, 66.4)
- moved R41 0.21 mm to (131.6, 66.4)
- moved R37 0.15 mm to (132.5, 66.4)
- moved C53 0.14 mm to (133.5, 66.4)
- moved R36 0.11 mm to (135.3, 66.3)
- moved C54 0.11 mm to (134.4, 66.4)
- moved C52 0.06 mm to (126.4, 74.4)
Routing:
- net +5V: track 22.3 -> 19.8 mm, vias 12 -> 14
- net /MCU/VDD: track 50.9 -> 48.6 mm
- net +9V: track 72.8 -> 73.9 mm
- net +5V_SYS: track 185.2 -> 185.7 mm
- net +3V3_SENS: track 99.2 -> 99.8 mm, vias 7 -> 6
- net GND: vias 237 -> 236
- added copper zone on F.Cu, net +5V
- added copper zone on F.Cu, net /MCU/VDD
