File: CAN.kicad_sch (KiCad schematic)
At the start: 7 parts, among them U12 SIT1051TK/3, U13 ZX-SH1.0-4PWT

Commit message: wip PDN
Connections:
- net CAN1_H: now also D6.1 (A1); no longer D6.2 (A2)
- net CAN1_L: now also D6.2 (A2); no longer D6.1 (A1)
Changed lines of the file:
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@@
+	)
+	(junction
+		(at 133.35 59.69)
+		(diameter 0)
+		(color 0 0 0 0)
 	)
 	(junction
@@
 	)
 	(junction
-		(at 133.35 72.39)
+		(at 128.27 72.39)
 		(diameter 0)
 		(color 0 0 0 0)
@@
 	(junction
 		(at 148.59 74.93)
-		(diameter 0)
-		(color 0 0 0 0)
-	)
-	(junction
-		(at 128.27 59.69)
 		(diameter 0)
 		(color 0 0 0 0)
@@
 	(wire
 		(pts
-			(xy 133.35 72.39) (xy 133.35 77.47)
+			(xy 133.35 59.69) (xy 133.35 77.47)
 		)
 		(stroke
@@
 	(wire
 		(pts
+			(xy 128.27 72.39) (xy 143.51 72.39)
+		)
+		(stroke
+			(width 0)
+			(type default)
+		)
+	)
+	(wire
+		(pts
 			(xy 146.05 68.58) (xy 149.86 68.58)
 		)
@@
 	(wire
 		(pts
-			(xy 133.35 72.39) (xy 143.51 72.39)
-		)
-		(stroke
-			(width 0)
-			(type default)
-		)
-	)
-	(wire
-		(pts
 			(xy 31.75 39.37) (xy 44.45 39.37)
 		)
@@
 	(wire
 		(pts
-			(xy 128.27 59.69) (xy 146.05 59.69)
+			(xy 120.65 59.69) (xy 133.35 59.69)
 		)
 		(stroke
@@
 	(wire
 		(pts
-			(xy 120.65 59.69) (xy 128.27 59.69)
-		)
-		(stroke
-			(width 0)
-			(type default)
-		)
-	)
-	(wire
-		(pts
-			(xy 128.27 59.69) (xy 128.27 77.47)
-		)
-		(stroke
-			(width 0)
-			(type default)
-		)
-	)
-	(wire
-		(pts
-			(xy 120.65 72.39) (xy 133.35 72.39)
-		)
-		(stroke
+			(xy 133.35 59.69) (xy 146.05 59.69)
+		)
+		(stroke
+			(width 0)
+			(type default)
+		)
+	)
+	(wire
+		(pts
+			(xy 120.65 72.39) (xy 128.27 72.39)
+		)
+		(stroke
+			(width 0)
+			(type default)
+		)
+	)
+	(wire
+		(pts
+			(xy 128.27 72.39) (xy 128.27 77.47)
+		)
+		(stroke
