File: POWER.kicad_sch (KiCad schematic)
At the start: 44 parts, among them U4 LMR43620R5RPER, U5 LMR604303SRAKRQ1, U6 AP7361C-33FGE-7, U7 AP7361C-33FGE-7

Commit message: labels
Parts:
- R19, R20: value 100K -> 10K
Changed lines of the file:
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@@
 			)
 		)
-		(property "Value" "100K"
+		(property "Value" "10K"
 			(at 218.44 67.31 0)
 			(show_name no)
@@
 			)
 		)
-		(property "Value" "100K"
+		(property "Value" "10K"
 			(at 218.44 123.19 0)
 			(show_name no)
