File: LEVIA_H7.kicad_sch (KiCad schematic)
At the start: 8 parts, among them U1 USBLC6-2P6

Commit message: BOM complete and JLC prod files generated
Parts:
- R1, R2: LCSC (none) -> C25905
- U1: LCSC (none) -> C2682291
- USB1: LCSC (none) -> C2894899
Changed lines of the file:
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@@
+			)
+		)
+		(property "LCSC" "C25905"
+			(at 72.39 45.72 90)
+			(hide yes)
+			(show_name no)
+			(do_not_autoplace no)
+			(effects
+				(font
+					(size 1.27 1.27)
+				)
 			)
 		)
@@
 		)
 		(property "LCSC Part" "C25905"
+			(at 72.39 48.26 90)
+			(hide yes)
+			(show_name no)
+			(do_not_autoplace no)
+			(effects
+				(font
+					(size 1.27 1.27)
+				)
+			)
+		)
+		(property "LCSC" "C25905"
 			(at 72.39 48.26 90)
 			(hide yes)
@@
 			)
 		)
+		(property "LCSC" "C2894899"
+			(at 53.34 55.88 0)
+			(hide yes)
+			(show_name no)
+			(do_not_autoplace no)
+			(effects
+				(font
+					(size 1.27 1.27)
+				)
+			)
+		)
 		(pin "B12"
 		)
@@
 			(at 90.17 55.88 0)
 			(hide yes)
+			(show_name no)
+			(do_not_autoplace no)
+			(effects
+				(font
+					(size 1.27 1.27)
+				)
+			)
+		)
+		(property "LCSC" "C2682291"
+			(at 90.17 55.88 0)
+			(hide yes)

Commit message: nextpcb manufacturing files updated
Parts:
- R1, R2: MPN (none) -> 0402WGF5101TCE; Manufacturer (none) -> UNI-ROYAL(Uniroyal Elec)
- U1: MPN (none) -> TPUSBLC6-2P6; Manufacturer (none) -> TECH PUBLIC
- USB1: MPN (none) -> HC-TYPE-C-16P-01M; Manufacturer (none) -> HCTL
Changed lines of the file:
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@@
+			)
+		)
+		(property "MPN" "0402WGF5101TCE"
+			(at 72.39 45.72 90)
+			(hide yes)
+			(show_name no)
+			(do_not_autoplace no)
+			(effects
+				(font
+					(size 1.27 1.27)
+				)
+			)
+		)
+		(property "Manufacturer" "UNI-ROYAL(Uniroyal Elec)"
+			(at 72.39 45.72 90)
+			(hide yes)
+			(show_name no)
+			(do_not_autoplace no)
+			(effects
+				(font
+					(size 1.27 1.27)
+				)
 			)
 		)
@@
 		)
 		(property "LCSC" "C25905"
+			(at 72.39 48.26 90)
+			(hide yes)
+			(show_name no)
+			(do_not_autoplace no)
+			(effects
+				(font
+					(size 1.27 1.27)
+				)
+			)
+		)
+		(property "MPN" "0402WGF5101TCE"
+			(at 72.39 48.26 90)
+			(hide yes)
+			(show_name no)
+			(do_not_autoplace no)
+			(effects
+				(font
+					(size 1.27 1.27)
+				)
+			)
+		)
+		(property "Manufacturer" "UNI-ROYAL(Uniroyal Elec)"
 			(at 72.39 48.26 90)
 			(hide yes)
@@
 			)
 		)
+		(property "MPN" "HC-TYPE-C-16P-01M"
+			(at 53.34 55.88 0)
+			(hide yes)
+			(show_name no)
+			(do_not_autoplace no)
+			(effects
+				(font
+					(size 1.27 1.27)
+				)
+			)
+		)
+		(property "Manufacturer" "HCTL"
+			(at 53.34 55.88 0)
+			(hide yes)
+			(show_name no)
+			(do_not_autoplace no)
+			(effects
+				(font
+					(size 1.27 1.27)
+				)
+			)
+		)
 		(pin "B12"
 		)
@@
 			(at 90.17 55.88 0)
 			(hide yes)
+			(show_name no)
+			(do_not_autoplace no)
+			(effects
+				(font
+					(size 1.27 1.27)
+				)
+			)
+		)
+		(property "MPN" "TPUSBLC6-2P6"
+			(at 90.17 55.88 0)
+			(hide yes)
+			(show_name no)
+			(do_not_autoplace no)
+			(effects
+				(font
+					(size 1.27 1.27)
+				)
+			)
+		)
+		(property "Manufacturer" "TECH PUBLIC"
+			(at 90.17 55.88 0)
+			(hide yes)

Commit message: DFA first round
Parts:
- U1: footprint Package_TO_SOT_SMD:SOT-666 -> EasyEDA:SOT-666-6_L1.6-W1.2-P0.50-LS1.6-BL
Changed lines of the file:
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@@
 			)
 		)
-		(property "Footprint" "Package_TO_SOT_SMD:SOT-666"
+		(property "Footprint" "EasyEDA:SOT-666-6_L1.6-W1.2-P0.50-LS1.6-BL"
 			(at 91.186 62.611 0)
 			(hide yes)
