File: MOTORS[1-4].kicad_sch (KiCad schematic)
At the start: 13 parts, among them U22 ZX-SH1.0-8PWT

Commit message: BOM complete and JLC prod files generated
Parts:
- R42, R43, R44, R45: LCSC (none) -> C25077
- U22: LCSC (none) -> C7430450
Changed lines of the file:
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@@
+			)
+		)
+		(property "LCSC" "C25077"
+			(at 78.74 60.96 90)
+			(hide yes)
+			(show_name no)
+			(do_not_autoplace no)
+			(effects
+				(font
+					(size 1.27 1.27)
+				)
 			)
 		)
@@
 			)
 		)
+		(property "LCSC" "C25077"
+			(at 78.74 66.04 90)
+			(hide yes)
+			(show_name no)
+			(do_not_autoplace no)
+			(effects
+				(font
+					(size 1.27 1.27)
+				)
+			)
+		)
 		(pin "2"
 		)
@@
 		)
 		(property "LCSC Part" "C25077"
+			(at 78.74 68.58 90)
+			(hide yes)
+			(show_name no)
+			(do_not_autoplace no)
+			(effects
+				(font
+					(size 1.27 1.27)
+				)
+			)
+		)
+		(property "LCSC" "C25077"
 			(at 78.74 68.58 90)
 			(hide yes)
@@
 			)
 		)
+		(property "LCSC" "C25077"
+			(at 78.74 63.5 90)
+			(hide yes)
+			(show_name no)
+			(do_not_autoplace no)
+			(effects
+				(font
+					(size 1.27 1.27)
+				)
+			)
+		)
 		(pin "2"
 		)
@@
 			(hide yes)
 			(show_name no)
+			(do_not_autoplace no)
+			(effects
+				(font
+					(size 1.27 1.27)
+				)
+			)
+		)
+		(property "LCSC" "C7430450"
+			(at 121.92 59.69 0)
+			(hide yes)
+			(show_name no)

Commit message: nextpcb manufacturing files updated
Parts:
- R42, R43, R44, R45: MPN (none) -> 0402WGF100JTCE; Manufacturer (none) -> UNI-ROYAL(Uniroyal Elec)
Changed lines of the file:
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@@
+			)
+		)
+		(property "MPN" "0402WGF100JTCE"
+			(at 78.74 60.96 90)
+			(hide yes)
+			(show_name no)
+			(do_not_autoplace no)
+			(effects
+				(font
+					(size 1.27 1.27)
+				)
+			)
+		)
+		(property "Manufacturer" "UNI-ROYAL(Uniroyal Elec)"
+			(at 78.74 60.96 90)
+			(hide yes)
+			(show_name no)
+			(do_not_autoplace no)
+			(effects
+				(font
+					(size 1.27 1.27)
+				)
 			)
 		)
@@
 			)
 		)
+		(property "MPN" "0402WGF100JTCE"
+			(at 78.74 66.04 90)
+			(hide yes)
+			(show_name no)
+			(do_not_autoplace no)
+			(effects
+				(font
+					(size 1.27 1.27)
+				)
+			)
+		)
+		(property "Manufacturer" "UNI-ROYAL(Uniroyal Elec)"
+			(at 78.74 66.04 90)
+			(hide yes)
+			(show_name no)
+			(do_not_autoplace no)
+			(effects
+				(font
+					(size 1.27 1.27)
+				)
+			)
+		)
 		(pin "2"
 		)
@@
 		)
 		(property "LCSC" "C25077"
+			(at 78.74 68.58 90)
+			(hide yes)
+			(show_name no)
+			(do_not_autoplace no)
+			(effects
+				(font
+					(size 1.27 1.27)
+				)
+			)
+		)
+		(property "MPN" "0402WGF100JTCE"
+			(at 78.74 68.58 90)
+			(hide yes)
+			(show_name no)
+			(do_not_autoplace no)
+			(effects
+				(font
+					(size 1.27 1.27)
+				)
+			)
+		)
+		(property "Manufacturer" "UNI-ROYAL(Uniroyal Elec)"
 			(at 78.74 68.58 90)
 			(hide yes)
@@
 			(at 78.74 63.5 90)
 			(hide yes)
+			(show_name no)
+			(do_not_autoplace no)
+			(effects
+				(font
+					(size 1.27 1.27)
+				)
+			)
+		)
+		(property "MPN" "0402WGF100JTCE"
+			(at 78.74 63.5 90)
+			(hide yes)
+			(show_name no)
+			(do_not_autoplace no)
+			(effects
+				(font
+					(size 1.27 1.27)
+				)
+			)
+		)
+		(property "Manufacturer" "UNI-ROYAL(Uniroyal Elec)"
+			(at 78.74 63.5 90)
+			(hide yes)

Commit message: DFA first round
Parts:
- TP10, TP3, TP4, TP5, TP6, TP7, TP8, TP9: now fitted
Changed lines of the file:
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@@
 		(exclude_from_sim no)
 		(in_bom no)
-		(on_board no)
-		(in_pos_files yes)
-		(dnp yes)
+		(on_board yes)
+		(in_pos_files yes)
+		(dnp no)
 		(property "Reference" "TP5"
 			(at 88.9 78.74 90)
@@
 		(exclude_from_sim no)
 		(in_bom no)
-		(on_board no)
-		(in_pos_files yes)
-		(dnp yes)
+		(on_board yes)
+		(in_pos_files yes)
+		(dnp no)
 		(property "Reference" "TP9"
 			(at 107.95 50.8 90)
@@
 		(exclude_from_sim no)
 		(in_bom no)
-		(on_board no)
-		(in_pos_files yes)
-		(dnp yes)
+		(on_board yes)
+		(in_pos_files yes)
+		(dnp no)
 		(property "Reference" "TP3"
 			(at 95.25 55.88 90)
@@
 		(exclude_from_sim no)
 		(in_bom no)
-		(on_board no)
-		(in_pos_files yes)
-		(dnp yes)
+		(on_board yes)
+		(in_pos_files yes)
+		(dnp no)
 		(property "Reference" "TP4"
 			(at 95.25 58.42 90)
@@
 		(exclude_from_sim no)
 		(in_bom no)
-		(on_board no)
-		(in_pos_files yes)
-		(dnp yes)
+		(on_board yes)
+		(in_pos_files yes)
+		(dnp no)
 		(property "Reference" "TP7"
 			(at 93.98 78.74 90)
@@
 		(exclude_from_sim no)
 		(in_bom no)
-		(on_board no)
-		(in_pos_files yes)
-		(dnp yes)
+		(on_board yes)
+		(in_pos_files yes)
+		(dnp no)
 		(property "Reference" "TP10"
 			(at 107.95 74.93 90)
@@
 		(exclude_from_sim no)
 		(in_bom no)
-		(on_board no)
-		(in_pos_files yes)
-		(dnp yes)
+		(on_board yes)
+		(in_pos_files yes)
+		(dnp no)
 		(property "Reference" "TP8"
 			(at 96.52 78.74 90)
@@
 		(exclude_from_sim no)
 		(in_bom no)
-		(on_board no)
-		(in_pos_files yes)
-		(dnp yes)
+		(on_board yes)
+		(in_pos_files yes)
+		(dnp no)
 		(property "Reference" "TP6"
 			(at 91.44 78.74 90)
